Commit message: feat(description): Robonine 팔 체인을 걷어내고 SO-101 체인 + ggao50 그리퍼로 교체
평행그리퍼 형상만 가져오려던 것이 팔 체인 규약까지 바꿔 놓은 상태였다.
Robonine 그리퍼를 안 쓰기로 했으므로 팔 체인도 검증된 SO-101 로 되돌린다.

- third_party/robonine, meshes/robonine, generate_parallel_arm_xacro.py 제거
- third_party/so_arm_101 신설. 상류 TheRobotStudio SO-ARM100/101(Apache-2.0)
  형상에 로컬 JD-AMR 실기에서 검증된 오리진·한계를 쓴다. NOTICE 로 출처 명시
- 관절 이름을 shoulder_pan/shoulder_lift/elbow_flex/wrist_flex/wrist_roll 로
  되돌려 capstone_pick/kinematics.py 와 규약을 맞춘다
- ggao50 은 상류에 라이선스 표기가 없어 메시를 벤더링하지 않는다. 배포된 STL
  실측 치수로 만든 단순 형상 프록시를 urdf/ggao50_gripper.xacro 에 둔다
- tool0, bottle_tcp, cup_tcp 프레임 추가. finger2_joint 가 finger1_joint 를 mimic
- 감사 스크립트 3종의 관절 이름·기대 집합을 새 규약에 맞춘다. 간섭 감사에서
  형상 없는 프레임이 KeyError 를 내던 버그도 고친다

감사 결과
- 붓기 관절 한계: fail -> pass. elbow 한계가 [0, 3.316] 에서 ±1.69 로 바뀌어
  붓기 자세의 -0.396 rad 이 정상 범위에 든다
- zero 자세 간섭: 충돌 18쌍 -> 0쌍, 교차 여유 18.78 -> 75.60 mm,
  팔↔LiDAR 4.33 -> 28.83 mm, 마스트 반경 31.36 -> 91.66 mm
- URDF 품질 감사와 고정 TF 검증 통과

남은 것
- 운반 후보 각도는 Robonine 체인용 legacy 값이라 SO-101 에서 양팔이 닿는다.
  새 체인과 tool0 기준으로 IK 재계산 필요
- 문서의 task 목표 좌표가 상수로 저장돼 있어 FK 산출값으로 대체해야 한다

Co-Authored-By: Claude Opus 5 (1M context) <noreply@anthropic.com>
Claude-Session: https://claude.ai/code/session_01Qya42b11SFUbRG5BmG5da4

File: src/hold_flow_description/urdf/hold_flow.urdf (robot description, URDF)
Before this commit: robot hold_flow, 35 links, 34 joints
Links:
- removed link left_clamp_1
- removed link left_clamp_2
- removed link left_link1_1
- removed link left_link2_1
- removed link left_link3_1
- removed link left_link4_1
- removed link left_link5_1
- removed link right_clamp_1
- removed link right_clamp_2
- removed link right_link1_1
- removed link right_link2_1
- removed link right_link3_1
- removed link right_link4_1
- removed link right_link5_1
- added link left_bottle_tcp, mass 1e-9
- added link left_cup_tcp, mass 1e-9
- added link left_finger1_link, mass 0.027; collision box size=0.031 0.072 0.050; visual box size=0.012 0.060 0.050
- added link left_finger2_link, mass 0.027; collision box size=0.031 0.072 0.050; visual box size=0.012 0.060 0.050
- added link left_gripper_base_link, mass 0.105; collision box size=0.1288 0.068 0.0725; visual box size=0.060 0.015 0.032
- added link left_gripper_link, mass 0.087; collision mesh filename=package://hold_flow_description/meshes/so101/sts3215_03a_v1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; collision mesh filename=package://hold_flow_description/meshes/so101/wrist_roll_fol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
- added link left_lower_arm_link, mass 0.104; collision mesh filename=package://hold_flow_description/meshes/so101/motor_holder_s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; collision mesh filename=package://hold_flow_description/meshes/so101/sts3215_03a_v1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
- added link left_shoulder_link, mass 0.100006; collision mesh filename=package://hold_flow_description/meshes/so101/motor_holder_s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; collision mesh filename=package://hold_flow_description/meshes/so101/rotation_pitch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
- added link left_tool0, mass 1e-9
- added link left_upper_arm_link, mass 0.103; collision mesh filename=package://hold_flow_description/meshes/so101/sts3215_03a_v1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; collision mesh filename=package://hold_flow_description/meshes/so101/upper_arm_so10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
- added link left_wrist_link, mass 0.079; collision mesh filename=package://hold_flow_description/meshes/so101/sts3215_03a_no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; collision mesh filename=package://hold_flow_description/meshes/so101/wrist_roll_pit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
- added link right_bottle_tcp, mass 1e-9
- added link right_cup_tcp, mass 1e-9
- added link right_finger1_link, mass 0.027; collision box size=0.031 0.072 0.050; visual box size=0.012 0.060 0.050
- added link right_finger2_link, mass 0.027; collision box size=0.031 0.072 0.050; visual box size=0.012 0.060 0.050
- added link right_gripper_base_link, mass 0.105; collision box size=0.1288 0.068 0.0725; visual box size=0.060 0.015 0.032
- added link right_gripper_link, mass 0.087; collision mesh filename=package://hold_flow_description/meshes/so101/sts3215_03a_v1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; collision mesh filename=package://hold_flow_description/meshes/so101/wrist_roll_fol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
- added link right_lower_arm_link, mass 0.104; collision mesh filename=package://hold_flow_description/meshes/so101/motor_holder_s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; collision mesh filename=package://hold_flow_description/meshes/so101/sts3215_03a_v1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
- added link right_shoulder_link, mass 0.100006; collision mesh filename=package://hold_flow_description/meshes/so101/motor_holder_s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; collision mesh filename=package://hold_flow_description/meshes/so101/rotation_pitch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
- added link right_tool0, mass 1e-9
- added link right_upper_arm_link, mass 0.103; collision mesh filename=package://hold_flow_description/meshes/so101/sts3215_03a_v1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; collision mesh filename=package://hold_flow_description/meshes/so101/upper_arm_so10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
- added link right_wrist_link, mass 0.079; collision mesh filename=package://hold_flow_description/meshes/so101/sts3215_03a_no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; collision mesh filename=package://hold_flow_description/meshes/so101/wrist_roll_pit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
- link left_base_link: geometry collision mesh filename=package://hold_flow_description/meshes/so101/base_motor_hol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; collision mesh filename=package://hold_flow_description/meshes/so101/base_so101_v2.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
- link right_base_link: geometry collision mesh filename=package://hold_flow_description/meshes/so101/base_motor_hol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; collision mesh filename=package://hold_flow_description/meshes/so101/base_so101_v2.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
Joints:
- removed joint left_base_link_to_link1
- removed joint left_left_clamp
- removed joint left_link1_to_link2
- removed joint left_link2_to_link3
- removed joint left_link3_to_link4
- removed joint left_link4_to_link5
- removed joint left_right_clamp
- removed joint right_base_link_to_link1
- removed joint right_left_clamp
- removed joint right_link1_to_link2
- removed joint right_link2_to_link3
- removed joint right_link3_to_link4
- removed joint right_link4_to_link5
- removed joint right_right_clamp
- added joint left_bottle_tcp_joint: type fixed, parent left_tool0, child left_bottle_tcp, origin xyz=0 0 0.09 rpy=0 0 0
- added joint left_cup_tcp_joint: type fixed, parent left_tool0, child left_cup_tcp, origin xyz=0 0 0.04 rpy=0 0 0
- added joint left_elbow_flex: type revolute, parent left_upper_arm_link, child left_lower_arm_link, origin xyz=-0.11257 -0.028 1.73763e-16 rpy=-3.63608e-16 8.74301e-16 1.5708, axis 0 0 1, limit lower=-1.69 upper=1.69 effort=10 velocity=10
- added joint left_finger1_joint: type prismatic, parent left_gripper_base_link, child left_finger1_link, origin xyz=0 -0.010 0 rpy=0 0 0, axis -1 0 0, limit lower=0.01 upper=0.0433 effort=40 velocity=0.05
- added joint left_finger2_joint: type prismatic, parent left_gripper_base_link, child left_finger2_link, origin xyz=0 -0.010 0 rpy=0 0 0, axis 1 0 0, limit lower=0.01 upper=0.0433 effort=40 velocity=0.05, mimic joint=left_finger1_joint multiplier=1.0 offset=0.0
- added joint left_gripper_mount_joint: type fixed, parent left_gripper_link, child left_gripper_base_link, origin xyz=-0.0079 -0.000218 0.0 rpy=1.5707963 0 0
- added joint left_shoulder_lift: type revolute, parent left_shoulder_link, child left_upper_arm_link, origin xyz=-0.0303992 -0.0182778 -0.0542 rpy=-1.5708 -1.5708 0, axis 0 0 1, limit lower=-1.74533 upper=1.74533 effort=10 velocity=10
- added joint left_shoulder_pan: type revolute, parent left_base_link, child left_shoulder_link, origin xyz=0.0388353 -8.97657e-09 0.0624 rpy=3.14159 4.18253e-17 -3.14159, axis 0 0 1, limit lower=-1.91986 upper=1.91986 effort=10 velocity=10
- added joint left_tool0_joint: type fixed, parent left_gripper_base_link, child left_tool0, origin xyz=0 -0.04 0 rpy=0 0 0
- added joint left_wrist_flex: type revolute, parent left_lower_arm_link, child left_wrist_link, origin xyz=-0.1349 0.0052 3.62355e-17 rpy=4.02456e-15 8.67362e-16 -1.5708, axis 0 0 1, limit lower=-1.65806 upper=1.65806 effort=10 velocity=10
- added joint left_wrist_roll: type revolute, parent left_wrist_link, child left_gripper_link, origin xyz=5.55112e-17 -0.0611 0.0181 rpy=1.5708 0.0486795 3.14159, axis 0 0 1, limit lower=-2.74385 upper=2.84121 effort=10 velocity=10
- added joint right_bottle_tcp_joint: type fixed, parent right_tool0, child right_bottle_tcp, origin xyz=0 0 0.09 rpy=0 0 0
- added joint right_cup_tcp_joint: type fixed, parent right_tool0, child right_cup_tcp, origin xyz=0 0 0.04 rpy=0 0 0
- added joint right_elbow_flex: type revolute, parent right_upper_arm_link, child right_lower_arm_link, origin xyz=-0.11257 -0.028 1.73763e-16 rpy=-3.63608e-16 8.74301e-16 1.5708, axis 0 0 1, limit lower=-1.69 upper=1.69 effort=10 velocity=10
- added joint right_finger1_joint: type prismatic, parent right_gripper_base_link, child right_finger1_link, origin xyz=0 -0.010 0 rpy=0 0 0, axis -1 0 0, limit lower=0.01 upper=0.0433 effort=40 velocity=0.05
- added joint right_finger2_joint: type prismatic, parent right_gripper_base_link, child right_finger2_link, origin xyz=0 -0.010 0 rpy=0 0 0, axis 1 0 0, limit lower=0.01 upper=0.0433 effort=40 velocity=0.05, mimic joint=right_finger1_joint multiplier=1.0 offset=0.0
- added joint right_gripper_mount_joint: type fixed, parent right_gripper_link, child right_gripper_base_link, origin xyz=-0.0079 -0.000218 0.0 rpy=1.5707963 0 0
- added joint right_shoulder_lift: type revolute, parent right_shoulder_link, child right_upper_arm_link, origin xyz=-0.0303992 -0.0182778 -0.0542 rpy=-1.5708 -1.5708 0, axis 0 0 1, limit lower=-1.74533 upper=1.74533 effort=10 velocity=10
- added joint right_shoulder_pan: type revolute, parent right_base_link, child right_shoulder_link, origin xyz=0.0388353 -8.97657e-09 0.0624 rpy=3.14159 4.18253e-17 -3.14159, axis 0 0 1, limit lower=-1.91986 upper=1.91986 effort=10 velocity=10
- added joint right_tool0_joint: type fixed, parent right_gripper_base_link, child right_tool0, origin xyz=0 -0.04 0 rpy=0 0 0
- added joint right_wrist_flex: type revolute, parent right_lower_arm_link, child right_wrist_link, origin xyz=-0.1349 0.0052 3.62355e-17 rpy=4.02456e-15 8.67362e-16 -1.5708, axis 0 0 1, limit lower=-1.65806 upper=1.65806 effort=10 velocity=10
- added joint right_wrist_roll: type revolute, parent right_wrist_link, child right_gripper_link, origin xyz=5.55112e-17 -0.0611 0.0181 rpy=1.5708 0.0486795 3.14159, axis 0 0 1, limit lower=-2.74385 upper=2.84121 effort=10 velocity=10

File: src/hold_flow_description/urdf/hold_flow.urdf.xacro (robot description, xacro)
@@ -4,9 +4,17 @@
   <xacro:include filename="$(find hold_flow_description)/urdf/mobile_base.xacro"/>
   <xacro:include filename="$(find hold_flow_description)/urdf/sensors.xacro"/>
-  <xacro:include filename="$(find hold_flow_description)/urdf/so101_parallel_arm.generated.xacro"/>
+  <xacro:include filename="$(find hold_flow_description)/third_party/so_arm_101/so101_arm.urdf.xacro"/>
+  <xacro:include filename="$(find hold_flow_description)/urdf/ggao50_gripper.xacro"/>
   <xacro:hold_flow_mobile_base/>
   <xacro:hold_flow_sensors/>
   <!-- 팔 베이스는 모두 250 mm 상판 경계 안에 있다. 좌우 이름은 MoveIt 그룹과 일치시킨다. -->
-  <xacro:so101_parallel_arm prefix="left_" parent="base_link" xyz="-0.065 0.070 0.0861" rpy="0 0 0"/>
-  <xacro:so101_parallel_arm prefix="right_" parent="base_link" xyz="-0.065 -0.070 0.0861" rpy="0 0 0"/>
+  <xacro:so101_arm prefix="left_" parent="base_link">
+    <origin xyz="-0.065 0.070 0.0861" rpy="0 0 0"/>
+  </xacro:so101_arm>
+  <xacro:so101_arm prefix="right_" parent="base_link">
+    <origin xyz="-0.065 -0.070 0.0861" rpy="0 0 0"/>
+  </xacro:so101_arm>
+  <!-- 상류 회전식 죠 대신 ggao50 평행 그리퍼를 손목 출력에 붙인다. -->
+  <xacro:ggao50_gripper prefix="left_" parent="left_gripper_link"/>
+  <xacro:ggao50_gripper prefix="right_" parent="right_gripper_link"/>
 </robot>

File: src/hold_flow_description/urdf/materials.xacro (robot description, xacro)
@@ -13,3 +13,15 @@
     <color rgba="0.63 0.66 0.70 1.0"/>
   </material>
+  <material name="so101_3d_printed">
+    <color rgba="0.16 0.17 0.19 1.0"/>
+  </material>
+  <material name="so101_sts3215">
+    <color rgba="0.10 0.10 0.12 1.0"/>
+  </material>
+  <material name="ggao50_printed">
+    <color rgba="0.75 0.77 0.80 1.0"/>
+  </material>
+  <material name="gripper_insert">
+    <color rgba="0.90 0.45 0.10 1.0"/>
+  </material>
 </robot>
