Commit message: feat(mechanical): 450×340 4분할 상판 모델로 전환

File: src/hold_flow_description/urdf/hold_flow.urdf (robot description, URDF)
Before this commit: robot hold_flow, 46 links, 45 joints
Links:
- removed link chassis_bottom_link
- removed link chassis_middle_link
- removed link chassis_top_link
- removed link lidar_riser_link
- added link battery_mount_plate_link, mass 0.12; collision box size=0.18 0.12 0.006; visual mesh filename=package://hold_flow_description/meshes/cad/battery_mount_pl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 scale=0.001 0.001 0.001
- added link lidar_mount_plate_link, mass 0.035; collision box size=0.09 0.075 0.003; visual mesh filename=package://hold_flow_description/meshes/cad/lidar_mount_plat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 scale=0.001 0.001 0.001
- added link lower_front_rail_link, mass 0.216; collision box size=0.02 0.45 0.02; visual box size=0.02 0.45 0.02
- added link lower_left_rail_link, mass 0.144; collision box size=0.3 0.02 0.02; visual box size=0.3 0.02 0.02
- added link lower_rear_rail_link, mass 0.216; collision box size=0.02 0.45 0.02; visual box size=0.02 0.45 0.02
- added link lower_right_rail_link, mass 0.144; collision box size=0.3 0.02 0.02; visual box size=0.3 0.02 0.02
- added link tabletop_front_left_link, mass 0.17; collision box size=0.2197 0.2247 0.006; visual mesh filename=package://hold_flow_description/meshes/cad/tabletop_front_l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 scale=0.001 0.001 0.001
- added link tabletop_front_right_link, mass 0.17; collision box size=0.2197 0.2247 0.006; visual mesh filename=package://hold_flow_description/meshes/cad/tabletop_front_r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 scale=0.001 0.001 0.001
- added link tabletop_rear_left_link, mass 0.17; collision box size=0.1197 0.2247 0.006; visual mesh filename=package://hold_flow_description/meshes/cad/tabletop_rear_le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 scale=0.001 0.001 0.001
- added link tabletop_rear_right_link, mass 0.17; collision box size=0.1197 0.2247 0.006; visual mesh filename=package://hold_flow_description/meshes/cad/tabletop_rear_ri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 scale=0.001 0.001 0.001
- added link upper_front_rail_link, mass 0.216; collision box size=0.02 0.45 0.02; visual box size=0.02 0.45 0.02
- added link upper_left_rail_link, mass 0.144; collision box size=0.3 0.02 0.02; visual box size=0.3 0.02 0.02
- added link upper_rear_rail_link, mass 0.216; collision box size=0.02 0.45 0.02; visual box size=0.02 0.45 0.02
- added link upper_right_rail_link, mass 0.144; collision box size=0.3 0.02 0.02; visual box size=0.3 0.02 0.02
- added link upper_x_seam_support_link, mass 0.216; collision box size=0.02 0.45 0.02; visual box size=0.02 0.45 0.02
- added link upper_y_seam_support_link, mass 0.144; collision box size=0.3 0.02 0.02; visual box size=0.3 0.02 0.02
- link front_left_frame_column_link: mass 0.29 -> 0.304; geometry collision box size=0.02 0.02 0.634; visual mesh filename=package://hold_flow_description/meshes/cad/frame_column.stl scale=0.001 0.001 0.001
- link front_right_frame_column_link: mass 0.29 -> 0.304; geometry collision box size=0.02 0.02 0.634; visual mesh filename=package://hold_flow_description/meshes/cad/frame_column.stl scale=0.001 0.001 0.001
- link rear_left_frame_column_link: mass 0.29 -> 0.304; geometry collision box size=0.02 0.02 0.634; visual mesh filename=package://hold_flow_description/meshes/cad/frame_column.stl scale=0.001 0.001 0.001
- link rear_right_frame_column_link: mass 0.29 -> 0.304; geometry collision box size=0.02 0.02 0.634; visual mesh filename=package://hold_flow_description/meshes/cad/frame_column.stl scale=0.001 0.001 0.001
Joints:
- removed joint chassis_bottom_link_joint
- removed joint chassis_middle_link_joint
- removed joint chassis_top_link_joint
- removed joint lidar_riser_link_joint
- added joint battery_mount_plate_link_joint: type fixed, parent base_link, child battery_mount_plate_link, origin xyz=-0.040 0 0.0351 rpy=0 0 0
- added joint lidar_mount_plate_link_joint: type fixed, parent base_link, child lidar_mount_plate_link, origin xyz=0.100 0 0.1121 rpy=0 0 0
- added joint lower_front_rail_link_joint: type fixed, parent base_link, child lower_front_rail_link, origin xyz=0.160 0 0.0171 rpy=0 0 0
- added joint lower_left_rail_link_joint: type fixed, parent base_link, child lower_left_rail_link, origin xyz=0 0.215 0.0171 rpy=0 0 0
- added joint lower_rear_rail_link_joint: type fixed, parent base_link, child lower_rear_rail_link, origin xyz=-0.160 0 0.0171 rpy=0 0 0
- added joint lower_right_rail_link_joint: type fixed, parent base_link, child lower_right_rail_link, origin xyz=0 -0.215 0.0171 rpy=0 0 0
- added joint tabletop_front_left_link_joint: type fixed, parent base_link, child tabletop_front_left_link, origin xyz=0.06015 0.11265 0.6811 rpy=0 0 0
- added joint tabletop_front_right_link_joint: type fixed, parent base_link, child tabletop_front_right_link, origin xyz=0.06015 -0.11265 0.6811 rpy=0 0 0
- added joint tabletop_rear_left_link_joint: type fixed, parent base_link, child tabletop_rear_left_link, origin xyz=-0.11015 0.11265 0.6811 rpy=0 0 0
- added joint tabletop_rear_right_link_joint: type fixed, parent base_link, child tabletop_rear_right_link, origin xyz=-0.11015 -0.11265 0.6811 rpy=0 0 0
- added joint upper_front_rail_link_joint: type fixed, parent base_link, child upper_front_rail_link, origin xyz=0.160 0 0.6711 rpy=0 0 0
- added joint upper_left_rail_link_joint: type fixed, parent base_link, child upper_left_rail_link, origin xyz=0 0.215 0.6711 rpy=0 0 0
- added joint upper_rear_rail_link_joint: type fixed, parent base_link, child upper_rear_rail_link, origin xyz=-0.160 0 0.6711 rpy=0 0 0
- added joint upper_right_rail_link_joint: type fixed, parent base_link, child upper_right_rail_link, origin xyz=0 -0.215 0.6711 rpy=0 0 0
- added joint upper_x_seam_support_link_joint: type fixed, parent base_link, child upper_x_seam_support_link, origin xyz=-0.050 0 0.6711 rpy=0 0 0
- added joint upper_y_seam_support_link_joint: type fixed, parent base_link, child upper_y_seam_support_link, origin xyz=0 0 0.6711 rpy=0 0 0
- joint battery_link_joint: origin xyz=-0.040 0 0.0071 rpy=0 0 0 -> xyz=-0.040 0 0.0611 rpy=0 0 0
- joint front_left_frame_column_link_joint: origin xyz=0.130 0.130 0.0351 rpy=0 0 0 -> xyz=0.150 0.205 0.0271 rpy=0 0 0
- joint front_right_frame_column_link_joint: origin xyz=0.130 -0.130 0.0351 rpy=0 0 0 -> xyz=0.150 -0.205 0.0271 rpy=0 0 0
- joint left_arm_backing_link_joint: origin xyz=0 0.075 0.6871 rpy=0 0 0 -> xyz=0.020 0.075 0.6871 rpy=0 0 0
- joint left_mount_joint: origin xyz=0 0.075 0.6931 rpy=0 0 0 -> xyz=0.020 0.075 0.6931 rpy=0 0 0
- joint rear_left_frame_column_link_joint: origin xyz=-0.130 0.130 0.0351 rpy=0 0 0 -> xyz=-0.150 0.205 0.0271 rpy=0 0 0
- joint rear_right_frame_column_link_joint: origin xyz=-0.130 -0.130 0.0351 rpy=0 0 0 -> xyz=-0.150 -0.205 0.0271 rpy=0 0 0
- joint right_arm_backing_link_joint: origin xyz=0 -0.075 0.6871 rpy=0 0 0 -> xyz=0.020 -0.075 0.6871 rpy=0 0 0
- joint right_mount_joint: origin xyz=0 -0.075 0.6931 rpy=0 0 0 -> xyz=0.020 -0.075 0.6931 rpy=0 0 0

File: src/hold_flow_description/urdf/hold_flow.urdf.xacro (robot description, xacro)
@@ -9,10 +9,10 @@
   <xacro:hold_flow_mobile_base/>
   <xacro:hold_flow_sensors/>
-  <!-- 상판 윗면 720 mm + 어댑터 6 mm. 팔은 상판 중앙의 y=±75 mm에 둔다. -->
+  <!-- 전면 모서리 x=170 mm에서 150 mm 뒤(x=20 mm), 상판 윗면 + 어댑터 6 mm. -->
   <xacro:so101_arm prefix="left_" parent="base_link">
-    <origin xyz="0 0.075 0.6931" rpy="0 0 0"/>
+    <origin xyz="0.020 0.075 0.6931" rpy="0 0 0"/>
   </xacro:so101_arm>
   <xacro:so101_arm prefix="right_" parent="base_link">
-    <origin xyz="0 -0.075 0.6931" rpy="0 0 0"/>
+    <origin xyz="0.020 -0.075 0.6931" rpy="0 0 0"/>
   </xacro:so101_arm>
   <!-- P0: 왼팔은 기본 SO-101 죠, 오른팔은 ggao50 평행 그리퍼 프록시다. -->

File: src/hold_flow_description/urdf/mobile_base.xacro (robot description, xacro)
@@ -72,16 +72,29 @@
       <origin xyz="0 0 0.0329" rpy="0 0 0"/>
     </joint>
-    <xacro:cad_mesh_link name="chassis_bottom_link" parent="base_link" xyz="0 0 -0.0269" mesh="chassis_bottom.stl" mass="0.400" sx="0.300" sy="0.300" sz="0.048" material="hold_flow_dark"/>
-    <xacro:cad_mesh_link name="chassis_middle_link" parent="base_link" xyz="0 0 0.0291" mesh="chassis_middle.stl" mass="0.340" sx="0.300" sy="0.300" sz="0.006" material="hold_flow_white"/>
-    <xacro:cad_mesh_link name="chassis_top_link" parent="base_link" xyz="0 0 0.6791" mesh="chassis_top.stl" mass="0.424" sx="0.300" sy="0.300" sz="0.008" material="hold_flow_white"/>
-    <xacro:cad_mesh_link name="front_left_frame_column_link" parent="base_link" xyz="0.130 0.130 0.0351" mesh="frame_column.stl" mass="0.290" sx="0.020" sy="0.020" sz="0.644" material="silver"/>
-    <xacro:cad_mesh_link name="front_right_frame_column_link" parent="base_link" xyz="0.130 -0.130 0.0351" mesh="frame_column.stl" mass="0.290" sx="0.020" sy="0.020" sz="0.644" material="silver"/>
-    <xacro:cad_mesh_link name="rear_left_frame_column_link" parent="base_link" xyz="-0.130 0.130 0.0351" mesh="frame_column.stl" mass="0.290" sx="0.020" sy="0.020" sz="0.644" material="silver"/>
-    <xacro:cad_mesh_link name="rear_right_frame_column_link" parent="base_link" xyz="-0.130 -0.130 0.0351" mesh="frame_column.stl" mass="0.290" sx="0.020" sy="0.020" sz="0.644" material="silver"/>
-    <xacro:cad_mesh_link name="left_arm_backing_link" parent="base_link" xyz="0 0.075 0.6871" mesh="arm_adapter.stl" mass="0.058" sx="0.130" sy="0.070" sz="0.006" material="hold_flow_dark"/>
-    <xacro:cad_mesh_link name="right_arm_backing_link" parent="base_link" xyz="0 -0.075 0.6871" mesh="arm_adapter.stl" mass="0.058" sx="0.130" sy="0.070" sz="0.006" material="hold_flow_dark"/>
+    <!-- 하부와 상부는 같은 340(x)×450(y) mm 2020 프로파일 외곽이다. -->
+    <xacro:primitive_box_link name="lower_front_rail_link" parent="base_link" xyz="0.160 0 0.0171" mass="0.216" sx="0.020" sy="0.450" sz="0.020" material="silver"/>
+    <xacro:primitive_box_link name="lower_rear_rail_link" parent="base_link" xyz="-0.160 0 0.0171" mass="0.216" sx="0.020" sy="0.450" sz="0.020" material="silver"/>
+    <xacro:primitive_box_link name="lower_left_rail_link" parent="base_link" xyz="0 0.215 0.0171" mass="0.144" sx="0.300" sy="0.020" sz="0.020" material="silver"/>
+    <xacro:primitive_box_link name="lower_right_rail_link" parent="base_link" xyz="0 -0.215 0.0171" mass="0.144" sx="0.300" sy="0.020" sz="0.020" material="silver"/>
+    <xacro:primitive_box_link name="upper_front_rail_link" parent="base_link" xyz="0.160 0 0.6711" mass="0.216" sx="0.020" sy="0.450" sz="0.020" material="silver"/>
+    <xacro:primitive_box_link name="upper_rear_rail_link" parent="base_link" xyz="-0.160 0 0.6711" mass="0.216" sx="0.020" sy="0.450" sz="0.020" material="silver"/>
+    <xacro:primitive_box_link name="upper_left_rail_link" parent="base_link" xyz="0 0.215 0.6711" mass="0.144" sx="0.300" sy="0.020" sz="0.020" material="silver"/>
+    <xacro:primitive_box_link name="upper_right_rail_link" parent="base_link" xyz="0 -0.215 0.6711" mass="0.144" sx="0.300" sy="0.020" sz="0.020" material="silver"/>
+    <xacro:primitive_box_link name="upper_x_seam_support_link" parent="base_link" xyz="-0.050 0 0.6711" mass="0.216" sx="0.020" sy="0.450" sz="0.020" material="silver"/>
+    <xacro:primitive_box_link name="upper_y_seam_support_link" parent="base_link" xyz="0 0 0.6711" mass="0.144" sx="0.300" sy="0.020" sz="0.020" material="silver"/>
+    <xacro:cad_mesh_link name="tabletop_front_left_link" parent="base_link" xyz="0.06015 0.11265 0.6811" mesh="tabletop_front_left.stl" mass="0.170" sx="0.2197" sy="0.2247" sz="0.006" material="hold_flow_white"/>
+    <xacro:cad_mesh_link name="tabletop_front_right_link" parent="base_link" xyz="0.06015 -0.11265 0.6811" mesh="tabletop_front_right.stl" mass="0.170" sx="0.2197" sy="0.2247" sz="0.006" material="hold_flow_white"/>
+    <xacro:cad_mesh_link name="tabletop_rear_left_link" parent="base_link" xyz="-0.11015 0.11265 0.6811" mesh="tabletop_rear_left.stl" mass="0.170" sx="0.1197" sy="0.2247" sz="0.006" material="hold_flow_white"/>
+    <xacro:cad_mesh_link name="tabletop_rear_right_link" parent="base_link" xyz="-0.11015 -0.11265 0.6811" mesh="tabletop_rear_right.stl" mass="0.170" sx="0.1197" sy="0.2247" sz="0.006" material="hold_flow_white"/>
+    <xacro:cad_mesh_link name="front_left_frame_column_link" parent="base_link" xyz="0.150 0.205 0.0271" mesh="frame_column.stl" mass="0.304" sx="0.020" sy="0.020" sz="0.634" material="silver"/>
+    <xacro:cad_mesh_link name="front_right_frame_column_link" parent="base_link" xyz="0.150 -0.205 0.0271" mesh="frame_column.stl" mass="0.304" sx="0.020" sy="0.020" sz="0.634" material="silver"/>
+    <xacro:cad_mesh_link name="rear_left_frame_column_link" parent="base_link" xyz="-0.150 0.205 0.0271" mesh="frame_column.stl" mass="0.304" sx="0.020" sy="0.020" sz="0.634" material="silver"/>
+    <xacro:cad_mesh_link name="rear_right_frame_column_link" parent="base_link" xyz="-0.150 -0.205 0.0271" mesh="frame_column.stl" mass="0.304" sx="0.020" sy="0.020" sz="0.634" material="silver"/>
+    <xacro:cad_mesh_link name="left_arm_backing_link" parent="base_link" xyz="0.020 0.075 0.6871" mesh="arm_adapter.stl" mass="0.058" sx="0.130" sy="0.070" sz="0.006" material="hold_flow_dark"/>
+    <xacro:cad_mesh_link name="right_arm_backing_link" parent="base_link" xyz="0.020 -0.075 0.6871" mesh="arm_adapter.stl" mass="0.058" sx="0.130" sy="0.070" sz="0.006" material="hold_flow_dark"/>
     <xacro:cad_mesh_link name="camera_backing_link" parent="base_link" xyz="-0.120 0 0.6871" mesh="camera_backing.stl" mass="0.030" sx="0.055" sy="0.055" sz="0.008" material="hold_flow_dark"/>
-    <xacro:cad_mesh_link name="lidar_riser_link" parent="base_link" xyz="0.100 0 0.0351" mesh="lidar_riser.stl" mass="0.274" sx="0.065" sy="0.050" sz="0.080" material="hold_flow_dark"/>
-    <xacro:primitive_box_link name="battery_link" parent="base_link" xyz="-0.040 0 0.0071" mass="0.550" sx="0.140" sy="0.080" sz="0.040" material="hold_flow_blue"/>
+    <xacro:cad_mesh_link name="battery_mount_plate_link" parent="base_link" xyz="-0.040 0 0.0351" mesh="battery_mount_plate.stl" mass="0.120" sx="0.180" sy="0.120" sz="0.006" material="hold_flow_blue"/>
+    <xacro:cad_mesh_link name="lidar_mount_plate_link" parent="base_link" xyz="0.100 0 0.1121" mesh="lidar_mount_plate.stl" mass="0.035" sx="0.090" sy="0.075" sz="0.003" material="hold_flow_blue"/>
+    <xacro:primitive_box_link name="battery_link" parent="base_link" xyz="-0.040 0 0.0611" mass="0.550" sx="0.140" sy="0.080" sz="0.040" material="hold_flow_blue"/>
     <xacro:primitive_box_link name="electronics_link" parent="base_link" xyz="0.030 0 0.0571" mass="0.350" sx="0.160" sy="0.120" sz="0.040" material="hold_flow_dark"/>
     <link name="left_wheel_link">

Commit message: fix(mechanical): 양팔을 상판 좌우 끝에 배치

File: src/hold_flow_description/urdf/hold_flow.urdf (robot description, URDF)
Before this commit: robot hold_flow, 58 links, 57 joints
Joints:
- joint left_arm_backing_link_joint: origin xyz=0.020 0.075 0.6871 rpy=0 0 0 -> xyz=0.020 0.170 0.6871 rpy=0 0 0
- joint left_mount_joint: origin xyz=0.020 0.075 0.6931 rpy=0 0 0 -> xyz=0.020 0.170 0.6931 rpy=0 0 0
- joint right_arm_backing_link_joint: origin xyz=0.020 -0.075 0.6871 rpy=0 0 0 -> xyz=0.020 -0.170 0.6871 rpy=0 0 0
- joint right_mount_joint: origin xyz=0.020 -0.075 0.6931 rpy=0 0 0 -> xyz=0.020 -0.170 0.6931 rpy=0 0 0

File: src/hold_flow_description/urdf/hold_flow.urdf.xacro (robot description, xacro)
@@ -11,8 +11,8 @@
   <!-- 전면 모서리 x=170 mm에서 150 mm 뒤(x=20 mm), 상판 윗면 + 어댑터 6 mm. -->
   <xacro:so101_arm prefix="left_" parent="base_link">
-    <origin xyz="0.020 0.075 0.6931" rpy="0 0 0"/>
+    <origin xyz="0.020 0.170 0.6931" rpy="0 0 0"/>
   </xacro:so101_arm>
   <xacro:so101_arm prefix="right_" parent="base_link">
-    <origin xyz="0.020 -0.075 0.6931" rpy="0 0 0"/>
+    <origin xyz="0.020 -0.170 0.6931" rpy="0 0 0"/>
   </xacro:so101_arm>
   <!-- P0: 왼팔은 기본 SO-101 죠, 오른팔은 ggao50 평행 그리퍼 프록시다. -->

File: src/hold_flow_description/urdf/mobile_base.xacro (robot description, xacro)
@@ -91,6 +91,6 @@
     <xacro:cad_mesh_link name="rear_left_frame_column_link" parent="base_link" xyz="-0.150 0.205 0.0271" mesh="frame_column.stl" mass="0.304" sx="0.020" sy="0.020" sz="0.634" material="silver"/>
     <xacro:cad_mesh_link name="rear_right_frame_column_link" parent="base_link" xyz="-0.150 -0.205 0.0271" mesh="frame_column.stl" mass="0.304" sx="0.020" sy="0.020" sz="0.634" material="silver"/>
-    <xacro:cad_mesh_link name="left_arm_backing_link" parent="base_link" xyz="0.020 0.075 0.6871" mesh="arm_adapter.stl" mass="0.058" sx="0.130" sy="0.070" sz="0.006" material="hold_flow_dark"/>
-    <xacro:cad_mesh_link name="right_arm_backing_link" parent="base_link" xyz="0.020 -0.075 0.6871" mesh="arm_adapter.stl" mass="0.058" sx="0.130" sy="0.070" sz="0.006" material="hold_flow_dark"/>
+    <xacro:cad_mesh_link name="left_arm_backing_link" parent="base_link" xyz="0.020 0.170 0.6871" mesh="arm_adapter.stl" mass="0.058" sx="0.130" sy="0.070" sz="0.006" material="hold_flow_dark"/>
+    <xacro:cad_mesh_link name="right_arm_backing_link" parent="base_link" xyz="0.020 -0.170 0.6871" mesh="arm_adapter.stl" mass="0.058" sx="0.130" sy="0.070" sz="0.006" material="hold_flow_dark"/>
     <xacro:cad_mesh_link name="camera_backing_link" parent="base_link" xyz="-0.120 0 0.6871" mesh="camera_backing.stl" mass="0.030" sx="0.055" sy="0.055" sz="0.008" material="hold_flow_dark"/>
     <xacro:cad_mesh_link name="battery_mount_plate_link" parent="base_link" xyz="-0.040 0 0.0351" mesh="battery_mount_plate.stl" mass="0.120" sx="0.180" sy="0.120" sz="0.006" material="hold_flow_blue"/>
