Commit message: feat(model): 최종 4륜 구동과 모델 소비 경로 통합

File: src/hold_flow_description/urdf/hold_flow.urdf (robot description, URDF)
Before this commit: robot hold_flow, 58 links, 57 joints
Links:
- removed link front_caster_link
- removed link rear_caster_link
- added link rear_left_wheel_link, mass 0.11; collision cylinder length=0.03 radius=0.0329; visual cylinder length=0.03 radius=0.0329
- added link rear_right_wheel_link, mass 0.11; collision cylinder length=0.03 radius=0.0329; visual cylinder length=0.03 radius=0.0329
- link left_wheel_link: geometry collision cylinder length=0.03 radius=0.0329; visual cylinder length=0.03 radius=0.0329
- link right_wheel_link: geometry collision cylinder length=0.03 radius=0.0329; visual cylinder length=0.03 radius=0.0329
Joints:
- removed joint front_caster_joint
- removed joint rear_caster_joint
- added joint rear_left_wheel_joint: type continuous, parent base_link, child rear_left_wheel_link, origin xyz=-0.105 0.255 0 rpy=0 0 0, axis 0 1 0, limit effort=0.981 velocity=4.72
- added joint rear_right_wheel_joint: type continuous, parent base_link, child rear_right_wheel_link, origin xyz=-0.105 -0.255 0 rpy=0 0 0, axis 0 1 0, limit effort=0.981 velocity=4.72
- joint left_wheel_joint: origin xyz=0 0.160 0 rpy=0 0 0 -> xyz=0.105 0.255 0 rpy=0 0 0
- joint right_wheel_joint: origin xyz=0 -0.160 0 rpy=0 0 0 -> xyz=0.105 -0.255 0 rpy=0 0 0

File: src/hold_flow_description/urdf/mobile_base.xacro (robot description, xacro)
@@ -58,5 +58,6 @@
   </xacro:macro>
   <xacro:macro name="hold_flow_mobile_base">
-    <!-- v0.3은 차체 중심과 구동축 중심의 바닥 투영점을 동일하게 둔다. -->
+    <!-- 모델 원점은 차체 중심이다. 실차 전륜축 원점과의 변환은 mechanical_calibration.yaml에 둔다. -->
+    <xacro:property name="drive_config" value="${xacro.load_yaml('../config/mechanical_calibration.yaml')['drive']}"/>
     <link name="base_footprint"/>
     <link name="base_link">
@@ -98,40 +99,19 @@
     <xacro:primitive_box_link name="battery_link" parent="base_link" xyz="-0.040 0 0.0611" mass="0.550" sx="0.140" sy="0.080" sz="0.040" material="hold_flow_blue"/>
     <xacro:primitive_box_link name="electronics_link" parent="base_link" xyz="0.030 0 0.0571" mass="0.350" sx="0.160" sy="0.120" sz="0.040" material="hold_flow_dark"/>
-    <link name="left_wheel_link">
-      <xacro:wheel_inertial mass="0.110" radius="0.0329" width="0.020"/>
-      <visual><origin rpy="1.570796 0 0"/><geometry><cylinder radius="0.0329" length="0.020"/></geometry><material name="hold_flow_dark"/></visual>
-      <collision><origin rpy="1.570796 0 0"/><geometry><cylinder radius="0.0329" length="0.020"/></geometry></collision>
+    <xacro:drive_wheel name="left_wheel" x="${drive_config['front_axle_x_m']}" y="${drive_config['geometric_wheel_center_separation_m'] / 2}" config="${drive_config}"/>
+    <xacro:drive_wheel name="right_wheel" x="${drive_config['front_axle_x_m']}" y="${-drive_config['geometric_wheel_center_separation_m'] / 2}" config="${drive_config}"/>
+    <xacro:drive_wheel name="rear_left_wheel" x="${drive_config['rear_axle_x_m']}" y="${drive_config['geometric_wheel_center_separation_m'] / 2}" config="${drive_config}"/>
+    <xacro:drive_wheel name="rear_right_wheel" x="${drive_config['rear_axle_x_m']}" y="${-drive_config['geometric_wheel_center_separation_m'] / 2}" config="${drive_config}"/>
+  </xacro:macro>
+  <xacro:macro name="drive_wheel" params="name x y config">
+    <link name="${name}_link">
+      <xacro:wheel_inertial mass="${config['mass_each_kg']}" radius="${config['wheel_radius_m']}" width="${config['visual_width_m']}"/>
+      <visual><origin rpy="${pi / 2} 0 0"/><geometry><cylinder radius="${config['wheel_radius_m']}" length="${config['visual_width_m']}"/></geometry><material name="hold_flow_dark"/></visual>
+      <collision><origin rpy="${pi / 2} 0 0"/><geometry><cylinder radius="${config['wheel_radius_m']}" length="${config['visual_width_m']}"/></geometry></collision>
     </link>
-    <joint name="left_wheel_joint" type="continuous">
-      <parent link="base_link"/><child link="left_wheel_link"/>
-      <origin xyz="0 0.160 0" rpy="0 0 0"/><axis xyz="0 1 0"/>
-      <limit effort="0.981" velocity="4.72"/><dynamics damping="0.02" friction="0.02"/>
-    </joint>
-    <link name="right_wheel_link">
-      <xacro:wheel_inertial mass="0.110" radius="0.0329" width="0.020"/>
-      <visual><origin rpy="1.570796 0 0"/><geometry><cylinder radius="0.0329" length="0.020"/></geometry><material name="hold_flow_dark"/></visual>
-      <collision><origin rpy="1.570796 0 0"/><geometry><cylinder radius="0.0329" length="0.020"/></geometry></collision>
-    </link>
-    <joint name="right_wheel_joint" type="continuous">
-      <parent link="base_link"/><child link="right_wheel_link"/>
-      <origin xyz="0 -0.160 0" rpy="0 0 0"/><axis xyz="0 1 0"/>
-      <limit effort="0.981" velocity="4.72"/><dynamics damping="0.02" friction="0.02"/>
-    </joint>
-    <xacro:ball_caster name="front_caster" x="0.120"/>
-    <xacro:ball_caster name="rear_caster" x="-0.120"/>
-  </xacro:macro>
-  <!-- URDF의 고정 구는 볼 캐스터 접촉 프록시다. 자유 회전 마찰은 USD에서 조정한다. -->
-  <xacro:macro name="ball_caster" params="name x">
-    <link name="${name}_link">
-      <inertial>
-        <mass value="0.060"/>
-        <inertia ixx="3.75e-6" ixy="0" ixz="0" iyy="3.75e-6" iyz="0" izz="3.75e-6"/>
-      </inertial>
-      <visual><geometry><sphere radius="0.0125"/></geometry><material name="silver"/></visual>
-      <collision><geometry><sphere radius="0.0125"/></geometry></collision>
-    </link>
-    <joint name="${name}_joint" type="fixed">
+    <joint name="${name}_joint" type="continuous">
       <parent link="base_link"/><child link="${name}_link"/>
-      <origin xyz="${x} 0 -0.0204" rpy="0 0 0"/>
+      <origin xyz="${x} ${y} 0" rpy="0 0 0"/><axis xyz="0 1 0"/>
+      <limit effort="${config['joint_effort_nm']}" velocity="${config['joint_velocity_radps']}"/><dynamics damping="0.02" friction="0.02"/>
     </joint>
   </xacro:macro>

Commit message: fix(camera): 렌즈 높이를 상판 위 54cm로 갱신

File: src/hold_flow_description/urdf/hold_flow.urdf (robot description, URDF)
Before this commit: robot hold_flow, 58 links, 57 joints
Links:
- link camera_mast_link: geometry collision box size=0.020 0.020 0.530; visual box size=0.020 0.020 0.530
Joints:
- joint camera_mount_joint: origin xyz=-0.006383 0 0.253472 rpy=0 0.6108652382 0 -> xyz=-0.006383 0 0.543472 rpy=0 0.6108652382 0

File: src/hold_flow_description/urdf/sensors.xacro (robot description, xacro)
@@ -2,12 +2,14 @@
 <robot xmlns:xacro="http://www.ros.org/wiki/xacro">
   <xacro:macro name="hold_flow_sensors">
-    <!-- 20×20×240 mm 후방 중앙 마스트. 8 mm 보강판 위 z=728 mm에서 시작한다. -->
+    <!-- 후방 중앙 마스트의 시각 프록시. 높이 근거는 design/mechanical/hold_flow_mechanical_v0_3.yaml camera.mount를 따른다. -->
     <link name="camera_mast_link">
-      <xacro:box_inertial mass="0.044" x="0.020" y="0.020" z="0.240"/>
+      <!-- 실물 마스트 재질·질량은 미측정이므로 기존 명목 질량을 유지한다. -->
+      <xacro:box_inertial mass="0.044" x="0.020" y="0.020" z="0.530"/>
       <visual>
-        <geometry><mesh filename="package://hold_flow_description/meshes/cad/camera_mast_segment.stl" scale="0.001 0.001 0.001"/></geometry>
+        <origin xyz="0 0 0.265"/>
+        <geometry><box size="0.020 0.020 0.530"/></geometry>
         <material name="hold_flow_dark"/>
       </visual>
-      <collision><origin xyz="0 0 0.120"/><geometry><box size="0.020 0.020 0.240"/></geometry></collision>
+      <collision><origin xyz="0 0 0.265"/><geometry><box size="0.020 0.020 0.530"/></geometry></collision>
     </link>
     <joint name="camera_mast_joint" type="fixed">
@@ -26,6 +28,6 @@
     <joint name="camera_mount_joint" type="fixed">
       <parent link="camera_mast_link"/><child link="camera_link"/>
-      <!-- 광학 중심 (-110,0,970) mm를 만들도록 35도 하향 자세에서 역산한 본체 중심. -->
-      <origin xyz="-0.006383 0 0.253472" rpy="0 0.6108652382 0"/>
+      <!-- 광학 중심과 기존 자세의 본체 중심 관계는 design/mechanical/hold_flow_mechanical_v0_3.yaml camera를 따른다. -->
+      <origin xyz="-0.006383 0 0.543472" rpy="0 0.6108652382 0"/>
     </joint>
     <link name="camera_cradle_link">
