Commit message: feat(sim): 300mm 양팔 로봇 URDF와 Isaac 모델 추가

File: src/hold_flow_description/third_party/so_arm_101/so101_arm.urdf.xacro (robot description, xacro)
@@ -4,7 +4,10 @@
   관절 오리진과 한계는 로컬 JD-AMR 실기에서 검증된 값이다. 출처는 같은
   디렉터리의 NOTICE 를 본다.
+  TheRobotStudio/SO-ARM100 commit: eecbe3e0a9ebb23e25ad7b2759b03884c6660903
+  upstream SO101 URDF sha256: 3a65d2d35e68a8d2f0c2cc176d19b884506543c93ba72980145b80abe276022c
+  local calibrated input sha256: d80275f4b4313229001a55836529fdf2747917bb49fc6c8490195ff42f0d7634
   이 파일은 scripts/generate_so101_arm_xacro.py 가 생성한다. 직접 편집하지 않는다.
-  그리퍼는 여기에 없다. 상류 회전식 죠 대신 ggao50 평행 그리퍼를 쓰므로
-  urdf/ggao50_gripper.xacro 가 ${prefix}gripper_link 에 이어 붙는다.
+  그리퍼는 여기에 없다. 왼팔 기본 회전식 죠와 오른팔 ggao50 평행 그리퍼를
+  별도 Xacro가 ${prefix}gripper_link 에 이어 붙인다.
 -->
 <robot xmlns:xacro="http://www.ros.org/wiki/xacro">
@@ -271,4 +274,6 @@
       <axis xyz="0 0 1" />
       <limit effort="10" velocity="10" lower="-1.91986" upper="1.91986" />
+      <dynamics damping="0.08" friction="0.02" />
+      <safety_controller soft_lower_limit="-1.86986" soft_upper_limit="1.86986" k_position="30" k_velocity="3" />
     </joint>
     <joint name="${prefix}shoulder_lift" type="revolute">
@@ -278,4 +283,6 @@
       <axis xyz="0 0 1" />
       <limit effort="10" velocity="10" lower="-1.74533" upper="1.74533" />
+      <dynamics damping="0.08" friction="0.02" />
+      <safety_controller soft_lower_limit="-1.69533" soft_upper_limit="1.69533" k_position="30" k_velocity="3" />
     </joint>
     <joint name="${prefix}elbow_flex" type="revolute">
@@ -285,4 +292,6 @@
       <axis xyz="0 0 1" />
       <limit effort="10" velocity="10" lower="-1.69" upper="1.69" />
+      <dynamics damping="0.08" friction="0.02" />
+      <safety_controller soft_lower_limit="-1.64" soft_upper_limit="1.64" k_position="30" k_velocity="3" />
     </joint>
     <joint name="${prefix}wrist_flex" type="revolute">
@@ -292,4 +301,6 @@
       <axis xyz="0 0 1" />
       <limit effort="10" velocity="10" lower="-1.65806" upper="1.65806" />
+      <dynamics damping="0.08" friction="0.02" />
+      <safety_controller soft_lower_limit="-1.60806" soft_upper_limit="1.60806" k_position="30" k_velocity="3" />
     </joint>
     <joint name="${prefix}wrist_roll" type="revolute">
@@ -299,4 +310,6 @@
       <axis xyz="0 0 1" />
       <limit effort="10" velocity="10" lower="-2.74385" upper="2.84121" />
+      <dynamics damping="0.08" friction="0.02" />
+      <safety_controller soft_lower_limit="-2.69385" soft_upper_limit="2.79121" k_position="30" k_velocity="3" />
     </joint>
   </xacro:macro>

File: src/hold_flow_description/urdf/ggao50_gripper.xacro (robot description, xacro)
@@ -67,10 +67,5 @@
     </joint>
     <!-- 두 죠 사이 중앙의 파지 기준. IK 목표와 FK 대조는 이 프레임을 쓴다. -->
-    <link name="${prefix}tool0">
-      <inertial>
-        <mass value="1e-9"/>
-        <inertia ixx="1e-12" ixy="0" ixz="0" iyy="1e-12" iyz="0" izz="1e-12"/>
-      </inertial>
-    </link>
+    <link name="${prefix}tool0"/>
     <xacro:object_tcp prefix="${prefix}" name="bottle_tcp" offset="${bottle_cap_offset_z}"/>
     <xacro:object_tcp prefix="${prefix}" name="cup_tcp" offset="${cup_rim_offset_z}"/>
@@ -83,10 +78,5 @@
       <origin xyz="0 0 ${offset}" rpy="0 0 0"/>
     </joint>
-    <link name="${prefix}${name}">
-      <inertial>
-        <mass value="1e-9"/>
-        <inertia ixx="1e-12" ixy="0" ixz="0" iyy="1e-12" iyz="0" izz="1e-12"/>
-      </inertial>
-    </link>
+    <link name="${prefix}${name}"/>
   </xacro:macro>
   <xacro:macro name="ggao50_jaw" params="prefix side sign">
@@ -97,4 +87,8 @@
       <axis xyz="${sign} 0 0"/>
       <limit lower="${ggao50_jaw_min}" upper="${ggao50_jaw_max}" effort="40" velocity="0.05"/>
+      <dynamics damping="0.50" friction="0.10"/>
+      <safety_controller
+        soft_lower_limit="0.011" soft_upper_limit="0.0423"
+        k_position="30" k_velocity="3"/>
       <xacro:if value="${side == 'finger2'}">
         <mimic joint="${prefix}finger1_joint" multiplier="1.0" offset="0.0"/>

File: src/hold_flow_description/urdf/hold_flow.urdf (robot description, URDF)
Before this commit: robot hold_flow, 43 links, 42 joints
Links:
- removed link camera_mast_lower_link
- removed link camera_mast_middle_link
- removed link camera_mast_upper_link
- removed link left_bottle_tcp
- removed link left_finger1_link
- removed link left_finger2_link
- removed link left_gripper_base_link
- added link battery_link, mass 0.55; collision box size=0.14 0.08 0.04; visual box size=0.14 0.08 0.04
- added link camera_color_optical_frame
- added link camera_mast_link, mass 0.044; collision box size=0.020 0.020 0.240; visual mesh filename=package://hold_flow_description/meshes/cad/camera_mast_segm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 scale=0.001 0.001 0.001
- added link electronics_link, mass 0.35; collision box size=0.16 0.12 0.04; visual box size=0.16 0.12 0.04
- added link front_caster_link, mass 0.060; collision sphere radius=0.0125; visual sphere radius=0.0125
- added link front_left_frame_column_link, mass 0.29; collision box size=0.02 0.02 0.644; visual mesh filename=package://hold_flow_description/meshes/cad/frame_column.stl scale=0.001 0.001 0.001
- added link front_right_frame_column_link, mass 0.29; collision box size=0.02 0.02 0.644; visual mesh filename=package://hold_flow_description/meshes/cad/frame_column.stl scale=0.001 0.001 0.001
- added link left_moving_jaw_link, mass 0.012; collision box size=0.0181 0.0129 0.0203; collision box size=0.0200 0.0399 0.0480
- added link rear_left_frame_column_link, mass 0.29; collision box size=0.02 0.02 0.644; visual mesh filename=package://hold_flow_description/meshes/cad/frame_column.stl scale=0.001 0.001 0.001
- added link rear_right_frame_column_link, mass 0.29; collision box size=0.02 0.02 0.644; visual mesh filename=package://hold_flow_description/meshes/cad/frame_column.stl scale=0.001 0.001 0.001
- link base_link: mass 0.001 -> 0.250
- link camera_backing_link: mass 0.0561 -> 0.03; geometry collision box size=0.055 0.055 0.008; visual mesh filename=package://hold_flow_description/meshes/cad/camera_backing.s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 scale=0.001 0.001 0.001
- link camera_cradle_link: mass 0.0853 -> 0.085; geometry collision box size=0.065 0.182 0.030; visual mesh filename=package://hold_flow_description/meshes/cad/astra_cradle.stl scale=0.001 0.001 0.001
- link chassis_bottom_link: mass 0.3258 -> 0.4; geometry collision box size=0.3 0.3 0.048; visual mesh filename=package://hold_flow_description/meshes/cad/chassis_bottom.s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 scale=0.001 0.001 0.001
- link chassis_middle_link: mass 0.2654 -> 0.34; geometry collision box size=0.3 0.3 0.006; visual mesh filename=package://hold_flow_description/meshes/cad/chassis_middle.s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 scale=0.001 0.001 0.001
- link chassis_top_link: mass 0.617 -> 0.424; geometry collision box size=0.3 0.3 0.008; visual mesh filename=package://hold_flow_description/meshes/cad/chassis_top.stl scale=0.001 0.001 0.001
- link left_arm_backing_link: mass 0.0773 -> 0.058; geometry collision box size=0.13 0.07 0.006; visual mesh filename=package://hold_flow_description/meshes/cad/arm_adapter.stl scale=0.001 0.001 0.001
- link left_cup_tcp: mass 1e-9 -> None
- link left_tool0: mass 1e-9 -> None
- link lidar_riser_link: mass 0.0992 -> 0.274; geometry collision box size=0.065 0.05 0.08; visual mesh filename=package://hold_flow_description/meshes/cad/lidar_riser.stl scale=0.001 0.001 0.001
- link right_arm_backing_link: mass 0.0773 -> 0.058; geometry collision box size=0.13 0.07 0.006; visual mesh filename=package://hold_flow_description/meshes/cad/arm_adapter.stl scale=0.001 0.001 0.001
- link right_bottle_tcp: mass 1e-9 -> None
- link right_cup_tcp: mass 1e-9 -> None
- link right_tool0: mass 1e-9 -> None
Joints:
- removed joint camera_mast_lower_joint
- removed joint camera_mast_middle_joint
- removed joint camera_mast_upper_joint
- removed joint left_bottle_tcp_joint
- removed joint left_finger1_joint
- removed joint left_finger2_joint
- removed joint left_gripper_mount_joint
- added joint battery_link_joint: type fixed, parent base_link, child battery_link, origin xyz=-0.040 0 0.0071 rpy=0 0 0
- added joint camera_color_optical_joint: type fixed, parent camera_depth_optical_frame, child camera_color_optical_frame, origin xyz=0 0 0 rpy=0 0 0
- added joint camera_mast_joint: type fixed, parent base_link, child camera_mast_link, origin xyz=-0.120 0 0.6951 rpy=0 0 0
- added joint electronics_link_joint: type fixed, parent base_link, child electronics_link, origin xyz=0.030 0 0.0571 rpy=0 0 0
- added joint front_caster_joint: type fixed, parent base_link, child front_caster_link, origin xyz=0.12 0 -0.0204 rpy=0 0 0
- added joint front_left_frame_column_link_joint: type fixed, parent base_link, child front_left_frame_column_link, origin xyz=0.130 0.130 0.0351 rpy=0 0 0
- added joint front_right_frame_column_link_joint: type fixed, parent base_link, child front_right_frame_column_link, origin xyz=0.130 -0.130 0.0351 rpy=0 0 0
- added joint left_gripper: type revolute, parent left_gripper_link, child left_moving_jaw_link, origin xyz=0.0202 0.0188 -0.0234 rpy=1.5708 -5.24284e-08 -1.41553e-15, axis 0 0 1, limit lower=-0.174533 upper=1.74533 effort=10 velocity=10
- added joint rear_left_frame_column_link_joint: type fixed, parent base_link, child rear_left_frame_column_link, origin xyz=-0.130 0.130 0.0351 rpy=0 0 0
- added joint rear_right_frame_column_link_joint: type fixed, parent base_link, child rear_right_frame_column_link, origin xyz=-0.130 -0.130 0.0351 rpy=0 0 0
- joint camera_backing_link_joint: origin xyz=-0.170 0 0.0861 rpy=0 0 0 -> xyz=-0.120 0 0.6871 rpy=0 0 0
- joint camera_depth_optical_joint: origin xyz=0.055 0 0 rpy=-1.570796 0 -1.570796 -> xyz=0.020 0 0 rpy=-1.5707963268 0 -1.5707963268
- joint camera_mount_joint: origin xyz=-0.042132 0 0.294353 rpy=0 0.698132 0 -> xyz=-0.006383 0 0.253472 rpy=0 0.6108652382 0; parent camera_mast_upper_link -> camera_mast_link
- joint chassis_bottom_link_joint: origin xyz=-0.090 0 -0.0269 rpy=0 0 0 -> xyz=0 0 -0.0269 rpy=0 0 0
- joint chassis_middle_link_joint: origin xyz=-0.090 0 0.0291 rpy=0 0 0 -> xyz=0 0 0.0291 rpy=0 0 0
- joint chassis_top_link_joint: origin xyz=-0.090 0 0.0781 rpy=0 0 0 -> xyz=0 0 0.6791 rpy=0 0 0
- joint laser_joint: origin xyz=0 0 0.1321 rpy=0 0 0 -> xyz=0.100 0 0.1321 rpy=0 0 0
- joint left_arm_backing_link_joint: origin xyz=-0.065 0.070 0.0721 rpy=0 0 0 -> xyz=0 0.075 0.6871 rpy=0 0 0
- joint left_cup_tcp_joint: origin xyz=0 0 0.04 rpy=0 0 0 -> xyz=0 0 0 rpy=0 0 0
- joint left_mount_joint: origin xyz=-0.065 0.070 0.0861 rpy=0 0 0 -> xyz=0 0.075 0.6931 rpy=0 0 0
- joint left_tool0_joint: origin xyz=0 -0.04 0 rpy=0 0 0 -> xyz=-0.0079 -0.000218121 -0.0981274 rpy=0 3.14159 0; parent left_gripper_base_link -> left_gripper_link
- joint left_wheel_joint: origin xyz=0 0.135 0 rpy=0 0 0 -> xyz=0 0.160 0 rpy=0 0 0
- joint lidar_riser_link_joint: origin xyz=0 0 0.0861 rpy=0 0 0 -> xyz=0.100 0 0.0351 rpy=0 0 0
- joint rear_caster_joint: origin xyz=-0.195 0 -0.0204 rpy=0 0 0 -> xyz=-0.12 0 -0.0204 rpy=0 0 0
- joint right_arm_backing_link_joint: origin xyz=-0.065 -0.070 0.0721 rpy=0 0 0 -> xyz=0 -0.075 0.6871 rpy=0 0 0
- joint right_mount_joint: origin xyz=-0.065 -0.070 0.0861 rpy=0 0 0 -> xyz=0 -0.075 0.6931 rpy=0 0 0
- joint right_wheel_joint: origin xyz=0 -0.135 0 rpy=0 0 0 -> xyz=0 -0.160 0 rpy=0 0 0

File: src/hold_flow_description/urdf/hold_flow.urdf.xacro (robot description, xacro)
@@ -5,16 +5,17 @@
   <xacro:include filename="$(find hold_flow_description)/urdf/sensors.xacro"/>
   <xacro:include filename="$(find hold_flow_description)/third_party/so_arm_101/so101_arm.urdf.xacro"/>
+  <xacro:include filename="$(find hold_flow_description)/urdf/so101_stock_gripper.xacro"/>
   <xacro:include filename="$(find hold_flow_description)/urdf/ggao50_gripper.xacro"/>
   <xacro:hold_flow_mobile_base/>
   <xacro:hold_flow_sensors/>
-  <!-- 팔 베이스는 모두 250 mm 상판 경계 안에 있다. 좌우 이름은 MoveIt 그룹과 일치시킨다. -->
+  <!-- 상판 윗면 720 mm + 어댑터 6 mm. 팔은 상판 중앙의 y=±75 mm에 둔다. -->
   <xacro:so101_arm prefix="left_" parent="base_link">
-    <origin xyz="-0.065 0.070 0.0861" rpy="0 0 0"/>
+    <origin xyz="0 0.075 0.6931" rpy="0 0 0"/>
   </xacro:so101_arm>
   <xacro:so101_arm prefix="right_" parent="base_link">
-    <origin xyz="-0.065 -0.070 0.0861" rpy="0 0 0"/>
+    <origin xyz="0 -0.075 0.6931" rpy="0 0 0"/>
   </xacro:so101_arm>
-  <!-- 상류 회전식 죠 대신 ggao50 평행 그리퍼를 손목 출력에 붙인다. -->
-  <xacro:ggao50_gripper prefix="left_" parent="left_gripper_link"/>
+  <!-- P0: 왼팔은 기본 SO-101 죠, 오른팔은 ggao50 평행 그리퍼 프록시다. -->
+  <xacro:so101_stock_gripper prefix="left_" parent="left_gripper_link"/>
   <xacro:ggao50_gripper prefix="right_" parent="right_gripper_link"/>
 </robot>

File: src/hold_flow_description/urdf/mobile_base.xacro (robot description, xacro)
@@ -20,4 +20,21 @@
     </inertial>
   </xacro:macro>
+  <xacro:macro name="primitive_box_link" params="name parent xyz mass sx sy sz material">
+    <link name="${name}">
+      <inertial>
+        <mass value="${mass}"/>
+        <inertia
+          ixx="${mass * (sy * sy + sz * sz) / 12.0}" ixy="0" ixz="0"
+          iyy="${mass * (sx * sx + sz * sz) / 12.0}" iyz="0"
+          izz="${mass * (sx * sx + sy * sy) / 12.0}"/>
+      </inertial>
+      <visual><geometry><box size="${sx} ${sy} ${sz}"/></geometry><material name="${material}"/></visual>
+      <collision><geometry><box size="${sx} ${sy} ${sz}"/></geometry></collision>
+    </link>
+    <joint name="${name}_joint" type="fixed">
+      <parent link="${parent}"/><child link="${name}"/><origin xyz="${xyz}" rpy="0 0 0"/>
+    </joint>
+  </xacro:macro>
+  <!-- 시각은 설계 STL, 충돌은 Isaac Sim 접촉 안정성을 위한 보수적 볼록 박스다. -->
   <xacro:macro name="cad_mesh_link" params="name parent xyz mesh mass sx sy sz material">
     <link name="${name}">
@@ -30,7 +47,6 @@
       </visual>
       <collision>
-        <geometry>
-          <mesh filename="package://hold_flow_description/meshes/cad/${mesh}" scale="0.001 0.001 0.001"/>
-        </geometry>
+        <origin xyz="0 0 ${sz / 2.0}" rpy="0 0 0"/>
+        <geometry><box size="${sx} ${sy} ${sz}"/></geometry>
       </collision>
     </link>
@@ -42,10 +58,11 @@
   </xacro:macro>
   <xacro:macro name="hold_flow_mobile_base">
-    <!-- base_footprint는 차체 중심이 아니라 구동 바퀴축의 바닥 투영점이다. -->
+    <!-- v0.3은 차체 중심과 구동축 중심의 바닥 투영점을 동일하게 둔다. -->
     <link name="base_footprint"/>
     <link name="base_link">
       <inertial>
-        <mass value="0.001"/>
-        <inertia ixx="1e-6" ixy="0" ixz="0" iyy="1e-6" iyz="0" izz="1e-6"/>
+        <origin xyz="0 0 0.030" rpy="0 0 0"/>
+        <mass value="0.250"/>
+        <inertia ixx="0.001602" ixy="0" ixz="0" iyy="0.001602" iyz="0" izz="0.002604"/>
       </inertial>
     </link>
@@ -55,74 +72,43 @@
       <origin xyz="0 0 0.0329" rpy="0 0 0"/>
     </joint>
-    <!-- 차체 중심은 바퀴축보다 90 mm 뒤에 있다. 메시 원점은 각 부품 바닥면이다. -->
-    <xacro:cad_mesh_link
-      name="chassis_bottom_link" parent="base_link" xyz="-0.090 0 -0.0269"
-      mesh="chassis_bottom.stl" mass="0.3258" sx="0.250" sy="0.250" sz="0.048"
-      material="hold_flow_dark"/>
-    <xacro:cad_mesh_link
-      name="chassis_middle_link" parent="base_link" xyz="-0.090 0 0.0291"
-      mesh="chassis_middle.stl" mass="0.2654" sx="0.250" sy="0.250" sz="0.006"
-      material="hold_flow_white"/>
-    <xacro:cad_mesh_link
-      name="chassis_top_link" parent="base_link" xyz="-0.090 0 0.0781"
-      mesh="chassis_top.stl" mass="0.6170" sx="0.250" sy="0.250" sz="0.008"
-      material="hold_flow_white"/>
-    <xacro:cad_mesh_link
-      name="left_arm_backing_link" parent="base_link" xyz="-0.065 0.070 0.0721"
-      mesh="arm_adapter.stl" mass="0.0773" sx="0.130" sy="0.090" sz="0.006"
-      material="hold_flow_dark"/>
-    <xacro:cad_mesh_link
-      name="right_arm_backing_link" parent="base_link" xyz="-0.065 -0.070 0.0721"
-      mesh="arm_adapter.stl" mass="0.0773" sx="0.130" sy="0.090" sz="0.006"
-      material="hold_flow_dark"/>
-    <xacro:cad_mesh_link
-      name="camera_backing_link" parent="base_link" xyz="-0.170 0 0.0861"
-      mesh="camera_backing.stl" mass="0.0561" sx="0.075" sy="0.075" sz="0.008"
-      material="hold_flow_dark"/>
-    <xacro:cad_mesh_link
-      name="lidar_riser_link" parent="base_link" xyz="0 0 0.0861"
-      mesh="lidar_riser.stl" mass="0.0992" sx="0.065" sy="0.050" sz="0.029"
-      material="hold_flow_dark"/>
+    <xacro:cad_mesh_link name="chassis_bottom_link" parent="base_link" xyz="0 0 -0.0269" mesh="chassis_bottom.stl" mass="0.400" sx="0.300" sy="0.300" sz="0.048" material="hold_flow_dark"/>
+    <xacro:cad_mesh_link name="chassis_middle_link" parent="base_link" xyz="0 0 0.0291" mesh="chassis_middle.stl" mass="0.340" sx="0.300" sy="0.300" sz="0.006" material="hold_flow_white"/>
+    <xacro:cad_mesh_link name="chassis_top_link" parent="base_link" xyz="0 0 0.6791" mesh="chassis_top.stl" mass="0.424" sx="0.300" sy="0.300" sz="0.008" material="hold_flow_white"/>
+    <xacro:cad_mesh_link name="front_left_frame_column_link" parent="base_link" xyz="0.130 0.130 0.0351" mesh="frame_column.stl" mass="0.290" sx="0.020" sy="0.020" sz="0.644" material="silver"/>
+    <xacro:cad_mesh_link name="front_right_frame_column_link" parent="base_link" xyz="0.130 -0.130 0.0351" mesh="frame_column.stl" mass="0.290" sx="0.020" sy="0.020" sz="0.644" material="silver"/>
+    <xacro:cad_mesh_link name="rear_left_frame_column_link" parent="base_link" xyz="-0.130 0.130 0.0351" mesh="frame_column.stl" mass="0.290" sx="0.020" sy="0.020" sz="0.644" material="silver"/>
+    <xacro:cad_mesh_link name="rear_right_frame_column_link" parent="base_link" xyz="-0.130 -0.130 0.0351" mesh="frame_column.stl" mass="0.290" sx="0.020" sy="0.020" sz="0.644" material="silver"/>
+    <xacro:cad_mesh_link name="left_arm_backing_link" parent="base_link" xyz="0 0.075 0.6871" mesh="arm_adapter.stl" mass="0.058" sx="0.130" sy="0.070" sz="0.006" material="hold_flow_dark"/>
+    <xacro:cad_mesh_link name="right_arm_backing_link" parent="base_link" xyz="0 -0.075 0.6871" mesh="arm_adapter.stl" mass="0.058" sx="0.130" sy="0.070" sz="0.006" material="hold_flow_dark"/>
+    <xacro:cad_mesh_link name="camera_backing_link" parent="base_link" xyz="-0.120 0 0.6871" mesh="camera_backing.stl" mass="0.030" sx="0.055" sy="0.055" sz="0.008" material="hold_flow_dark"/>
+    <xacro:cad_mesh_link name="lidar_riser_link" parent="base_link" xyz="0.100 0 0.0351" mesh="lidar_riser.stl" mass="0.274" sx="0.065" sy="0.050" sz="0.080" material="hold_flow_dark"/>
+    <xacro:primitive_box_link name="battery_link" parent="base_link" xyz="-0.040 0 0.0071" mass="0.550" sx="0.140" sy="0.080" sz="0.040" material="hold_flow_blue"/>
+    <xacro:primitive_box_link name="electronics_link" parent="base_link" xyz="0.030 0 0.0571" mass="0.350" sx="0.160" sy="0.120" sz="0.040" material="hold_flow_dark"/>
     <link name="left_wheel_link">
       <xacro:wheel_inertial mass="0.110" radius="0.0329" width="0.020"/>
-      <visual>
-        <origin rpy="1.570796 0 0"/>
-        <geometry><cylinder radius="0.0329" length="0.020"/></geometry>
-        <material name="hold_flow_dark"/>
-      </visual>
-      <collision>
-        <origin rpy="1.570796 0 0"/>
-        <geometry><cylinder radius="0.0329" length="0.020"/></geometry>
-      </collision>
+      <visual><origin rpy="1.570796 0 0"/><geometry><cylinder radius="0.0329" length="0.020"/></geometry><material name="hold_flow_dark"/></visual>
+      <collision><origin rpy="1.570796 0 0"/><geometry><cylinder radius="0.0329" length="0.020"/></geometry></collision>
     </link>
     <joint name="left_wheel_joint" type="continuous">
-      <parent link="base_link"/>
-      <child link="left_wheel_link"/>
-      <origin xyz="0 0.135 0" rpy="0 0 0"/>
-      <axis xyz="0 1 0"/>
-      <limit effort="0.981" velocity="4.72"/>
-      <dynamics damping="0.02" friction="0.02"/>
+      <parent link="base_link"/><child link="left_wheel_link"/>
+      <origin xyz="0 0.160 0" rpy="0 0 0"/><axis xyz="0 1 0"/>
+      <limit effort="0.981" velocity="4.72"/><dynamics damping="0.02" friction="0.02"/>
     </joint>
     <link name="right_wheel_link">
       <xacro:wheel_inertial mass="0.110" radius="0.0329" width="0.020"/>
-      <visual>
-        <origin rpy="1.570796 0 0"/>
-        <geometry><cylinder radius="0.0329" length="0.020"/></geometry>
-        <material name="hold_flow_dark"/>
-      </visual>
-      <collision>
-        <origin rpy="1.570796 0 0"/>
-        <geometry><cylinder radius="0.0329" length="0.020"/></geometry>
-      </collision>
+      <visual><origin rpy="1.570796 0 0"/><geometry><cylinder radius="0.0329" length="0.020"/></geometry><material name="hold_flow_dark"/></visual>
+      <collision><origin rpy="1.570796 0 0"/><geometry><cylinder radius="0.0329" length="0.020"/></geometry></collision>
     </link>
     <joint name="right_wheel_joint" type="continuous">
-      <parent link="base_link"/>
-      <child link="right_wheel_link"/>
-      <origin xyz="0 -0.135 0" rpy="0 0 0"/>
-      <axis xyz="0 1 0"/>
-      <limit effort="0.981" velocity="4.72"/>
-      <dynamics damping="0.02" friction="0.02"/>
+      <parent link="base_link"/><child link="right_wheel_link"/>
+      <origin xyz="0 -0.160 0" rpy="0 0 0"/><axis xyz="0 1 0"/>
+      <limit effort="0.981" velocity="4.72"/><dynamics damping="0.02" friction="0.02"/>
     </joint>
-    <link name="rear_caster_link">
+    <xacro:ball_caster name="front_caster" x="0.120"/>
+    <xacro:ball_caster name="rear_caster" x="-0.120"/>
+  </xacro:macro>
+  <!-- URDF의 고정 구는 볼 캐스터 접촉 프록시다. 자유 회전 마찰은 USD에서 조정한다. -->
+  <xacro:macro name="ball_caster" params="name x">
+    <link name="${name}_link">
       <inertial>
         <mass value="0.060"/>
@@ -132,8 +118,7 @@
       <collision><geometry><sphere radius="0.0125"/></geometry></collision>
     </link>
-    <joint name="rear_caster_joint" type="fixed">
-      <parent link="base_link"/>
-      <child link="rear_caster_link"/>
-      <origin xyz="-0.195 0 -0.0204" rpy="0 0 0"/>
+    <joint name="${name}_joint" type="fixed">
+      <parent link="base_link"/><child link="${name}_link"/>
+      <origin xyz="${x} 0 -0.0204" rpy="0 0 0"/>
     </joint>
   </xacro:macro>
