Commit message: feat(sim): 300mm 양팔 로봇 URDF와 Isaac 모델 추가

File: src/hold_flow_description/urdf/sensors.xacro (robot description, xacro)
@@ -2,31 +2,16 @@
 <robot xmlns:xacro="http://www.ros.org/wiki/xacro">
   <xacro:macro name="hold_flow_sensors">
-    <!-- 마스트 중심: 차체 (-80, 0), base_footprint 기준 (-170, 0). -->
-    <link name="camera_mast_lower_link">
-      <xacro:box_inertial mass="0.1773" x="0.045" y="0.035" z="0.267"/>
-      <visual><geometry><mesh filename="package://hold_flow_description/meshes/cad/camera_mast_segment.stl" scale="0.001 0.001 0.001"/></geometry><material name="hold_flow_dark"/></visual>
-      <collision><geometry><box size="0.045 0.035 0.267"/></geometry><origin xyz="0 0 0.1335"/></collision>
+    <!-- 20×20×240 mm 후방 중앙 마스트. 8 mm 보강판 위 z=728 mm에서 시작한다. -->
+    <link name="camera_mast_link">
+      <xacro:box_inertial mass="0.044" x="0.020" y="0.020" z="0.240"/>
+      <visual>
+        <geometry><mesh filename="package://hold_flow_description/meshes/cad/camera_mast_segment.stl" scale="0.001 0.001 0.001"/></geometry>
+        <material name="hold_flow_dark"/>
+      </visual>
+      <collision><origin xyz="0 0 0.120"/><geometry><box size="0.020 0.020 0.240"/></geometry></collision>
     </link>
-    <joint name="camera_mast_lower_joint" type="fixed">
-      <parent link="base_link"/><child link="camera_mast_lower_link"/>
-      <origin xyz="-0.170 0 0.0941" rpy="0 0 0"/>
-    </joint>
-    <link name="camera_mast_middle_link">
-      <xacro:box_inertial mass="0.1773" x="0.045" y="0.035" z="0.267"/>
-      <visual><geometry><mesh filename="package://hold_flow_description/meshes/cad/camera_mast_segment.stl" scale="0.001 0.001 0.001"/></geometry><material name="hold_flow_dark"/></visual>
-      <collision><geometry><box size="0.045 0.035 0.267"/></geometry><origin xyz="0 0 0.1335"/></collision>
-    </link>
-    <joint name="camera_mast_middle_joint" type="fixed">
-      <parent link="camera_mast_lower_link"/><child link="camera_mast_middle_link"/>
-      <origin xyz="0 0 0.207" rpy="0 0 0"/>
-    </joint>
-    <link name="camera_mast_upper_link">
-      <xacro:box_inertial mass="0.1497" x="0.045" y="0.035" z="0.267"/>
-      <visual><geometry><mesh filename="package://hold_flow_description/meshes/cad/camera_mast_segment.stl" scale="0.001 0.001 0.001"/></geometry><material name="hold_flow_dark"/></visual>
-      <collision><geometry><box size="0.045 0.035 0.267"/></geometry><origin xyz="0 0 0.1335"/></collision>
-    </link>
-    <joint name="camera_mast_upper_joint" type="fixed">
-      <parent link="camera_mast_middle_link"/><child link="camera_mast_upper_link"/>
-      <origin xyz="0 0 0.207" rpy="0 0 0"/>
+    <joint name="camera_mast_joint" type="fixed">
+      <parent link="base_link"/><child link="camera_mast_link"/>
+      <origin xyz="-0.120 0 0.6951" rpy="0 0 0"/>
     </joint>
     <link name="camera_link">
@@ -35,27 +20,32 @@
         <inertia ixx="0.00076283" ixy="0" ixz="0" iyy="0.00010085" iyz="0" izz="0.00074465"/>
       </inertial>
-      <!-- Astra S 실제 외곽 165(W)×48(H)×40(D) mm: +X 깊이, +Y 폭, +Z 높이. -->
+      <!-- Astra S: +X 깊이, +Y 폭, +Z 높이. 본체 프레임은 질량중심 근사다. -->
       <visual><geometry><box size="0.040 0.165 0.048"/></geometry><material name="hold_flow_blue"/></visual>
       <collision><geometry><box size="0.040 0.165 0.048"/></geometry></collision>
     </link>
     <joint name="camera_mount_joint" type="fixed">
-      <parent link="camera_mast_upper_link"/><child link="camera_link"/>
-      <!-- 광학 중심이 차체 (-80, 0, 800) mm가 되도록 55 mm 전면 오프셋을 역산. -->
-      <origin xyz="-0.042132 0 0.294353" rpy="0 0.698132 0"/>
+      <parent link="camera_mast_link"/><child link="camera_link"/>
+      <!-- 광학 중심 (-110,0,970) mm를 만들도록 35도 하향 자세에서 역산한 본체 중심. -->
+      <origin xyz="-0.006383 0 0.253472" rpy="0 0.6108652382 0"/>
     </joint>
     <link name="camera_cradle_link">
-      <xacro:box_inertial mass="0.0853" x="0.065" y="0.182" z="0.030"/>
+      <xacro:box_inertial mass="0.085" x="0.065" y="0.182" z="0.030"/>
       <visual><geometry><mesh filename="package://hold_flow_description/meshes/cad/astra_cradle.stl" scale="0.001 0.001 0.001"/></geometry><material name="hold_flow_dark"/></visual>
-      <collision><geometry><mesh filename="package://hold_flow_description/meshes/cad/astra_cradle.stl" scale="0.001 0.001 0.001"/></geometry></collision>
+      <collision><origin xyz="0 0 0.015"/><geometry><box size="0.065 0.182 0.030"/></geometry></collision>
     </link>
     <joint name="camera_cradle_joint" type="fixed">
       <parent link="camera_link"/><child link="camera_cradle_link"/>
-      <!-- 거치대 바닥 상면 z=6 mm에 카메라 하단이 닿도록 본체 중심에서 30 mm 하향. -->
       <origin xyz="0 0 -0.030" rpy="0 0 0"/>
     </joint>
+    <!-- Astra 계열 optical convention: +Z forward, +X right, +Y down. -->
     <link name="camera_depth_optical_frame"/>
     <joint name="camera_depth_optical_joint" type="fixed">
       <parent link="camera_link"/><child link="camera_depth_optical_frame"/>
-      <origin xyz="0.055 0 0" rpy="-1.570796 0 -1.570796"/>
+      <origin xyz="0.020 0 0" rpy="-1.5707963268 0 -1.5707963268"/>
+    </joint>
+    <link name="camera_color_optical_frame"/>
+    <joint name="camera_color_optical_joint" type="fixed">
+      <parent link="camera_depth_optical_frame"/><child link="camera_color_optical_frame"/>
+      <origin xyz="0 0 0" rpy="0 0 0"/>
     </joint>
     <link name="laser_link">
@@ -69,6 +59,5 @@
     <joint name="laser_joint" type="fixed">
       <parent link="base_link"/><child link="laser_link"/>
-      <!-- 차체 x=90 mm는 바퀴축 기준 x=0, 바닥 z=165 mm는 base_link 기준 132.1 mm. -->
-      <origin xyz="0 0 0.1321" rpy="0 0 0"/>
+      <origin xyz="0.100 0 0.1321" rpy="0 0 0"/>
     </joint>
   </xacro:macro>
