Commit message: fix(navigation): 근접 재주차 회전과 마지막 면 정렬 수정

File: src/navigation/jdamr_cube_description/urdf/new_base_real.urdf (robot description, URDF)
Before this commit: robot new_base_real, 14 links, 13 joints
Joints:
- joint camera_mount_joint: origin xyz=-0.275 0 0.540 rpy=0.011934068034722573 0.41246669799099545 -0.0007507445375463481 -> xyz=-0.275 0 0.540 rpy=-0.03011453253432204 0.5837829655386328 -0.0007507445375463481

Commit message: fix(navigation): 도크 직진 이탈과 사륜 충돌 외곽 반영

File: src/navigation/jdamr_cube_description/urdf/new_base_real.urdf (robot description, URDF)
Before this commit: robot new_base_real, 14 links, 13 joints
Links:
- removed link rear_left_caster_contact_projection
- removed link rear_right_caster_contact_projection
- added link rear_left_wheel_link; collision cylinder length=0.030 radius=0.0329; visual cylinder length=0.030 radius=0.0329
- added link rear_right_wheel_link; collision cylinder length=0.030 radius=0.0329; visual cylinder length=0.030 radius=0.0329
Joints:
- removed joint rear_left_caster_contact_joint
- removed joint rear_right_caster_contact_joint
- added joint rear_left_wheel_joint: type continuous, parent base_link, child rear_left_wheel_link, origin xyz=-0.210 0.255 0.0329 rpy=0 0 0, axis 0 1 0
- added joint rear_right_wheel_joint: type continuous, parent base_link, child rear_right_wheel_link, origin xyz=-0.210 -0.255 0.0329 rpy=0 0 0, axis 0 1 0

Commit message: fix(navigation): 카메라 각도 변경과 깊이 평면 자세 반영

File: src/navigation/jdamr_cube_description/urdf/new_base_real.urdf (robot description, URDF)
Before this commit: robot new_base_real, 14 links, 13 joints
Joints:
- joint camera_mount_joint: origin xyz=-0.275 0 0.540 rpy=-0.03011453253432204 0.5837829655386328 -0.0007507445375463481 -> xyz=-0.275 0 0.540 rpy=-0.01946375975958315 0.639563761794311 -0.0007507445375463481

Commit message: fix(navigation): 근접 보정과 후면 재관측 흐름 수정

File: src/navigation/jdamr_cube_description/urdf/new_base_real.urdf (robot description, URDF)
Before this commit: robot new_base_real, 14 links, 13 joints
Joints:
- joint camera_mount_joint: origin xyz=-0.275 0 0.540 rpy=-0.01946375975958315 0.639563761794311 -0.0007507445375463481 -> xyz=-0.275 0 0.540 rpy=-0.039023134986489794 0.9171698002732518 -0.0007507445375463481

Commit message: fix(navigation): 도크 접근과 이동 경계의 지연 및 입력 회복 개선 (#75)
* fix(navigation): 출발 지연 경로와 주차 실행 결과 판정 수정

* fix(navigation): 근접 재주차 회전과 마지막 면 정렬 수정

* docs(navigation): 재주차 회전 오류와 수정본 주행 결과 기록

* fix(navigation): 실측 기준 책상 면 보정과 최종 접근 속도 조정

* docs(navigation): 책상 면 보정과 양측 12mm 실측 기록

* fix(navigation): 급수대 경유와 연속 정밀접근 및 테이블 점유 후보 반영

* docs(navigation): 연속 접근 수정본의 파이 반영 근거 기록

* fix(navigation): 평행한 3센치 도크 배치와 테이블 킵아웃 동기화

* fix(navigation): 이동 중 면 안정화 복구와 미세 정렬 감속 적용

* fix(navigation): 깊이 입력 지연을 작업 종료 대신 정지 대기로 복구

* docs(navigation): 관측 지연 수정과 주행 중지 및 남은 구간 기록

* fix(navigation): 미세 회전 감속을 통합하고 반대 보정 전 면 재관측 적용

* fix(navigation): 도크 지도 오차 재접근과 깊이 면 재획득 복구

* docs(navigation): 실물 주차 오차와 급수대 이탈 충돌 기록

* fix(navigation): 도크 직진 이탈과 사륜 충돌 외곽 반영

* fix(navigation): 도크 이탈의 중복 전역 경로 검사 제거

* fix(navigation): 주차 재개 지연과 도크 반복 조향 개선

* fix(navigation): 도크 뒤쪽 기존 킵아웃 겹침에서 직진 이탈 허용

* fix(navigation): 고정 테이블 탐색과 연속 주차의 반복 동작 개선

* feat(navigation): 라이다 후면 박스 정밀주차와 평면 추적 추가

* docs(navigation): 메모리 실측과 알고리즘 전환 보류 근거 기록

* fix(navigation): 중복 준비 조회 제거와 실제 카메라 대기 계측

* fix(navigation): 도크 복귀를 후면 라이다 정밀주차로 연결

* fix(navigation): 근접 도크에서 감시형 직선 이탈 연결

* fix(navigation): 도크 접근과 이동 경계의 지연 및 입력 회복 개선

* fix(navigation): 주차 초과 접근 보정과 복귀 이동점 판정 분리

* fix(navigation): 카메라 각도 변경과 깊이 평면 자세 반영

* fix(navigation): 근접 책상 검출과 최종 거리 재확인 보정

* fix(navigation): 근접 보정과 후면 재관측 흐름 수정

* fix(navigation): 출발 기준 박스 중심으로 도크 복귀 보정

* fix(navigation): 급수대 근접 정렬과 재접근 차단 수정

* fix(navigation): 책상 관측 전진과 도크 초기화 복구 수정

* fix(navigation): 태스크 사이 고정 대기와 중복 정지 제거

---------

Co-authored-by: mmporong <mmporong@gmail.com>

File: src/navigation/jdamr_cube_description/urdf/new_base_real.urdf (robot description, URDF)
Before this commit: robot new_base_real, 14 links, 13 joints
Links:
- removed link rear_left_caster_contact_projection
- removed link rear_right_caster_contact_projection
- added link rear_left_wheel_link; collision cylinder length=0.030 radius=0.0329; visual cylinder length=0.030 radius=0.0329
- added link rear_right_wheel_link; collision cylinder length=0.030 radius=0.0329; visual cylinder length=0.030 radius=0.0329
Joints:
- removed joint rear_left_caster_contact_joint
- removed joint rear_right_caster_contact_joint
- added joint rear_left_wheel_joint: type continuous, parent base_link, child rear_left_wheel_link, origin xyz=-0.210 0.255 0.0329 rpy=0 0 0, axis 0 1 0
- added joint rear_right_wheel_joint: type continuous, parent base_link, child rear_right_wheel_link, origin xyz=-0.210 -0.255 0.0329 rpy=0 0 0, axis 0 1 0
- joint camera_mount_joint: origin xyz=-0.275 0 0.540 rpy=0.011934068034722573 0.41246669799099545 -0.0007507445375463481 -> xyz=-0.275 0 0.540 rpy=-0.039023134986489794 0.9171698002732518 -0.0007507445375463481

Commit message: fix(amr): 후면 도킹 각도와 근접 기억점 판정을 보정

File: src/navigation/jdamr_cube_description/urdf/new_base_real.urdf (robot description, URDF)
Before this commit: robot new_base_real, 14 links, 13 joints
Joints:
- joint laser_joint: origin xyz=-0.010 0 0.150 rpy=0 0 3.141592653589793 -> xyz=-0.010 0 0.150 rpy=0 0 3.202979549615386

Commit message: fix(amr): 주차 좌표와 카메라 자세 및 후면 접근 수정

File: src/navigation/jdamr_cube_description/urdf/new_base_real.urdf (robot description, URDF)
Before this commit: robot new_base_real, 14 links, 13 joints
Joints:
- joint camera_mount_joint: origin xyz=-0.275 0 0.540 rpy=-0.039023134986489794 0.9171698002732518 -0.0007507445375463481 -> xyz=-0.275 0 0.540 rpy=0.01837857145491081 0.8414714126967582 0.0
